File: ESP-SOCKET/Eagle/esp-socket-4.brd (EAGLE design)
At the start: 57.1 x 64.3 mm, 25 parts, among them K2 SRD-03VDC, Q1 BC847BSMD

Commit message: 0.0.1
Routing:
- net GND: track 130.9 -> 131.7 mm
Other:
- board text added: "2018"
- board text removed: "TSP-03"
